File: openmv_can_shield.kicad_sch (KiCad schematic)
At the start: 32 parts, among them J1 WAGO_250-204, J2 Pulse_JXD6-0001NL, J3 Conn_01x03, J4 Conn_01x02, J5 Conn_02x03_Odd_Even, J6 Conn_02x05_Odd_Even, J7 Conn_01x02, J8 Conn_01x02, Q1 BSS138, Q2 BSS138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

Commit message: Updated schematics and layout to have complete, DRC clean layout, Gerbers not updated
Parts:
- J3: footprint (none) -> Connector_PinHeader_2.54mm:PinHeader_1x03_P2.54mm_Vertical
Connections:
- net GND: now also J2.SH
- net ETH_RXN renamed ETH_RX_N
- net ETH_RXP renamed ETH_RX_P
- net ETH_TXN renamed ETH_TX_N
- net ETH_TXP renamed ETH_TX_P
- no-connect marks 16 -> 17
Changed lines of the file:
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@@
   (no_connect (at 142.875 152.4))
   (no_connect (at 142.875 144.78))
+  (no_connect (at 52.705 132.715))
   (no_connect (at 227.965 78.74))
   (no_connect (at 248.285 124.46))
@@
     (stroke (width 0) (type default) (color 0 0 0 0))
   )
+  (wire (pts (xy 250.825 154.94) (xy 250.825 157.48))
+    (stroke (width 0) (type default) (color 0 0 0 0))
+  )
   (wire (pts (xy 255.905 118.745) (xy 255.905 124.46))
     (stroke (width 0) (type default) (color 0 0 0 0))
@@
     (stroke (width 0) (type default) (color 0 0 0 0))
   )
+  (wire (pts (xy 52.705 127.635) (xy 65.405 127.635))
+    (stroke (width 0) (type default) (color 0 0 0 0))
+  )
   (wire (pts (xy 246.38 33.655) (xy 258.445 33.655))
     (stroke (width 0) (type default) (color 0 0 0 0))
@@
     (stroke (width 0) (type default) (color 0 0 0 0))
   )
-  (wire (pts (xy 52.705 120.015) (xy 62.23 120.015))
+  (wire (pts (xy 52.705 120.015) (xy 65.405 120.015))
     (stroke (width 0) (type default) (color 0 0 0 0))
   )
@@
     (stroke (width 0) (type default) (color 0 0 0 0))
   )
-  (wire (pts (xy 52.705 127.635) (xy 62.23 127.635))
-    (stroke (width 0) (type default) (color 0 0 0 0))
-  )
   (wire (pts (xy 115.57 147.32) (xy 130.175 147.32))
     (stroke (width 0) (type default) (color 0 0 0 0))
@@
     (stroke (width 0) (type default) (color 0 0 0 0))
   )
-  (wire (pts (xy 52.705 117.475) (xy 62.23 117.475))
+  (wire (pts (xy 52.705 117.475) (xy 65.405 117.475))
     (stroke (width 0) (type default) (color 0 0 0 0))
   )
@@
     (stroke (width 0) (type default) (color 0 0 0 0))
   )
-  (wire (pts (xy 52.705 125.095) (xy 62.23 125.095))
+  (wire (pts (xy 52.705 125.095) (xy 65.405 125.095))
     (stroke (width 0) (type default) (color 0 0 0 0))
   )
@@
     (stroke (width 0) (type default) (color 0 0 0 0))
   )
-  (wire (pts (xy 52.705 122.555) (xy 62.23 122.555))
+  (wire (pts (xy 52.705 122.555) (xy 65.405 122.555))
     (stroke (width 0) (type default) (color 0 0 0 0))
   )
@@
     (effects (font (size 1.27 1.27)) (justify right bottom))
   )
-  (label "ETH_TXP" (at 62.23 127.635 180)
+  (label "ETH_TX_P" (at 65.405 127.635 180)
     (effects (font (size 1.27 1.27)) (justify right bottom))
   )
@@
     (effects (font (size 1.27 1.27)) (justify left bottom))
   )
-  (label "ETH_TXN" (at 206.375 137.16 0)
-    (effects (font (size 1.27 1.27)) (justify left bottom))
-  )
-  (label "ETH_LED" (at 62.23 117.475 180)
+  (label "ETH_TX_N" (at 206.375 137.16 0)
+    (effects (font (size 1.27 1.27)) (justify left bottom))
+  )
+  (label "ETH_LED" (at 65.405 117.475 180)
     (effects (font (size 1.27 1.27)) (justify right bottom))
   )
@@
     (effects (font (size 1.27 1.27)) (justify right bottom))
   )
-  (label "ETH_RXN" (at 206.375 147.32 0)
+  (label "ETH_RX_N" (at 206.375 147.32 0)
     (effects (font (size 1.27 1.27)) (justify left bottom))
   )
@@
     (effects (font (size 1.27 1.27)) (justify right bottom))
   )
-  (label "ETH_RXN" (at 62.23 120.015 180)
+  (label "ETH_RX_N" (at 65.405 120.015 180)
     (effects (font (size 1.27 1.27)) (justify right bottom))
   )
@@
     (effects (font (size 1.27 1.27)) (justify left bottom))
   )
-  (label "ETH_TXP" (at 206.375 132.08 0)
+  (label "ETH_TX_P" (at 206.375 132.08 0)
     (effects (font (size 1.27 1.27)) (justify left bottom))
   )
@@
     (effects (font (size 1.27 1.27)) (justify left bottom))
   )
-  (label "ETH_RXP" (at 62.23 122.555 180)
-    (effects (font (size 1.27 1.27)) (justify right bottom))
-  )
-  (label "ETH_RXP" (at 206.375 142.24 0)
+  (label "ETH_RX_P" (at 65.405 122.555 180)
+    (effects (font (size 1.27 1.27)) (justify right bottom))
+  )
+  (label "ETH_RX_P" (at 206.375 142.24 0)
     (effects (font (size 1.27 1.27)) (justify left bottom))
   )
@@
     (effects (font (size 1.27 1.27)) (justify right bottom))
   )
-  (label "ETH_TXN" (at 62.23 125.095 180)
+  (label "ETH_TX_N" (at 65.405 125.095 180)
     (effects (font (size 1.27 1.27)) (justify right bottom))
   )
@@
       (effects (font (size 1.27 1.27)) (justify left))
     )
-    (property "Footprint" "" (id 2) (at 135.255 184.15 0)
+    (property "Footprint" "Connector_PinHeader_2.54mm:PinHeader_1x03_P2.54mm_Vertical" (id 2) (at 135.255 184.15 0)
       (effects (font (size 1.27 1.27)) hide)
     )
@@
     (pin "1")
   )
+  (symbol (lib_id "power:GND") (at 250.825 157.48 0) (unit 1)
+    (in_bom yes) (on_board yes)
+    (property "Reference" "#PWR0122" (id 0) (at 250.825 163.83 0)
+      (effects (font (size 1.27 1.27)) hide)
+    )
+    (property "Value" "GND" (id 1) (at 250.825 161.29 0))
+    (property "Footprint" "" (id 2) (at 250.825 157.48 0)
+      (effects (font (size 1.27 1.27)) hide)
+    )
+    (property "Datasheet" "" (id 3) (at 250.825 157.48 0)
+      (effects (font (size 1.27 1.27)) hide)
+    )
+    (pin "1")
+  )
   (symbol (lib_id "Connector_Generic:Conn_02x03_Odd_Even") (at 138.43 104.775 0) (unit 1)
     (in_bom yes) (on_board yes)
@@
       (reference "#PWR0121") (unit 1) (value "+3.3V") (footprint "")
     )
+    (path "/dc076562-fdbc-4462-8f40-9a8c52462afb"
+      (reference "#PWR0122") (unit 1) (value "GND") (footprint "")
+    )
     (path "/7b478b53-e149-47a6-a9f3-1795cd7fcc84"
